File: Tiny vr.kicad_pcb (KiCad board)
At the start: 2 copper layers, 22 x 37 mm, 17 parts, among them J1 USB_C_Receptacle_USB2.0_14P, J2 Conn_01x02_Pin, J3 Conn_01x08, Q1 AO3400A, U1 ESP32-S3-MINI-1, U2 LD1117S33TR_SOT223, U3 TP4057, U4 DW01A

Commit message: updated finished routing
Parts:
- moved R3 6.51 mm to (35.5, 59.5), turned to 90 degrees
- moved D1 6.27 mm to (30.0, 60.0), turned to -90 degrees
- moved D2 6.01 mm to (28.0, 60.0), turned to -90 degrees
- moved R2 4.92 mm to (30.0, 54.0)
- moved R5 4.30 mm to (36.0, 56.0), turned to 0 degrees
- moved R4 3.35 mm to (32.0, 59.5), turned to 90 degrees
- moved U4 1.87 mm to (39.6, 57.5), turned to 0 degrees
- moved J2 0.90 mm to (45.5, 35.0)
Connections:
- U1 pad 28: Net-(J3-Pin_3) -> unconnected-(U1-IO33-Pad28)
- U1 pad 29: Net-(J3-Pin_4) -> unconnected-(U1-IO34-Pad29)
- U1 pad 31: Net-(J3-Pin_5) -> Net-(J3-Pin_8)
- U1 pad 32: Net-(J3-Pin_6) -> Net-(J3-Pin_7)
- U1 pad 33: Net-(J3-Pin_7) -> Net-(J3-Pin_6)
- U1 pad 34: Net-(J3-Pin_8) -> Net-(J3-Pin_5)
- U1 pad 35: unconnected-(U1-IO39-Pad35) -> Net-(J3-Pin_4)
- U1 pad 36: unconnected-(U1-IO40-Pad36) -> Net-(J3-Pin_3)
Routing:
- net Net-(J1-SHIELD): track 0.35 -> 182.2 mm, vias 0 -> 2
- net Net-(J3-Pin_1): track 0.00 -> 66.2 mm, vias 0 -> 2
- net Net-(J2-Pin_1): track 0.07 -> 50.7 mm, vias 0 -> 2
- net Net-(U1-USB_D-): track 0.00 -> 30.2 mm
- net Net-(J2-Pin_2): track 0.00 -> 20.7 mm, vias 0 -> 1
- net Net-(J3-Pin_8): track 0.00 -> 19.2 mm
- net Net-(U3-V_{CC}): track 0.00 -> 18.4 mm, vias 0 -> 2
- net Net-(J3-Pin_7): track 0.00 -> 18.3 mm
- net Net-(U1-USB_D+): track 0.00 -> 18.2 mm
- net Net-(J3-Pin_6): track 0.00 -> 15.8 mm
- net Net-(J3-Pin_5): track 0.00 -> 13.6 mm
- net Net-(Q1-G): track 0.00 -> 13.5 mm
- net Net-(D1-A): track 0.00 -> 11.9 mm
- net Net-(J3-Pin_4): track 0.00 -> 11.9 mm
- net Net-(J3-Pin_3): track 0.00 -> 11.1 mm
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Other:
- board size 22 x 37 mm -> 22.5 x 37 mm
- board text removed: ":2vr"
